Commit message: added bc

File: assets/door.urdf (robot description, URDF)
Before this commit: robot two_leaf_door, 4 links, 3 joints
Links:
- link door_frame: geometry visual mesh filename=meshes/door_frame.stl scale=1 1 1

Commit message: finished act

File: assets/door.urdf (robot description, URDF)
Before this commit: robot two_leaf_door, 4 links, 3 joints
Links:
- link door_frame: geometry collision mesh filename=meshes/door_frame.stl scale=1 1 1; visual mesh filename=meshes/door_frame.stl scale=1 1 1
